Commit message: Refactoring out separate xacro files

File: src/rsj_description/urdf/rsj.xacro (robot description, xacro)
@@ -1,35 +1,9 @@
 <?xml version="1.0"?>
 <!-- Ros Simplest Joint Robot -->
-<robot name="rsj" xmlns:xacro="http://www.ros.org/wiki/xacro">
-  <!-- Constants for robot dimensions -->
-  <xacro:property name="PI" value="3.1415926535897931"/>
-  <xacro:property name="mass" value="1" /> <!-- arbitrary value for mass -->
-  <xacro:property name="width" value="0.1" /> <!-- Square dimensions (widthxwidth) of beams -->
-  <xacro:property name="height1" value="2" /> <!-- Link 1 -->
-  <xacro:property name="height2" value="1" /> <!-- Link 2 -->
-  <xacro:property name="axle_offset" value="0.05" /> <!-- Space btw top of beam and the each joint -->
-  <!-- Gazebo-customization elements, including Gazebo colors -->
-  <gazebo>
-    <plugin name="gazebo_ros_control" filename="libgazebo_ros_control.so">
-      <robotNamespace>/rsj</robotNamespace>
-      <robotSimType>gazebo_ros_control/DefaultRobotHWSim</robotSimType>
-    </plugin>
-  </gazebo>
-  <!-- Link1 -->
-  <gazebo reference="link1">
-    <material>Gazebo/Orange</material>
-  </gazebo>
-  <!-- Link2 -->
-  <gazebo reference="link2">
-    <mu1>0.2</mu1>
-    <mu2>0.2</mu2>
-    <material>Gazebo/Black</material>
-  </gazebo>
-  <material name="black">
-    <color rgba="0.0 0.0 0.0 1.0"/>
-  </material>
-  <material name="orange">
-    <color rgba="${255/255} ${108/255} ${10/255} 1.0"/>
-  </material>
+<robot name="rsj"
+  xmlns:xacro="http://www.ros.org/wiki/xacro">
+  <xacro:include filename="properties.xacro"/>
+  <xacro:include filename="gazebo.xacro"/>
+  <xacro:include filename="materials.xacro"/>
   <!-- Used for fixing robot to Gazebo 'base_link' -->
   <link name="world"/>
@@ -56,9 +30,6 @@
       <origin xyz="0 0 ${height1/2}" rpy="0 0 0"/>
       <mass value="${mass}"/>
-      <inertia
-        ixx="${mass / 12.0 * (width*width + height1*height1)}" ixy="0.0" ixz="0.0"
-        iyy="${mass / 12.0 * (height1*height1 + width*width)}" iyz="0.0"
-        izz="${mass / 12.0 * (width*width + width*width)}"/>
-      </inertial>
+      <inertia ixx="${mass / 12.0 * (width*width + height1*height1)}" ixy="0.0" ixz="0.0" iyy="${mass / 12.0 * (height1*height1 + width*width)}" iyz="0.0" izz="${mass / 12.0 * (width*width + width*width)}"/>
+    </inertial>
   </link>
   <joint name="joint1" type="continuous">
@@ -87,9 +58,6 @@
       <origin xyz="0 0 ${height2/2 - axle_offset}" rpy="0 0 0"/>
       <mass value="${mass}"/>
-      <inertia
-        ixx="${mass / 12.0 * (width*width + height2*height2)}" ixy="0.0" ixz="0.0"
-        iyy="${mass / 12.0 * (height2*height2 + width*width)}" iyz="0.0"
-        izz="${mass / 12.0 * (width*width + width*width)}"/>
-      </inertial>
+      <inertia ixx="${mass / 12.0 * (width*width + height2*height2)}" ixy="0.0" ixz="0.0" iyy="${mass / 12.0 * (height2*height2 + width*width)}" iyz="0.0" izz="${mass / 12.0 * (width*width + width*width)}"/>
+    </inertial>
   </link>
   <transmission name="tran1">
